File: scm-pcb.kicad_sch (KiCad schematic)
At the start: 8 parts, among them J1 Raspberry_Pi_2_3, U1 LM2596, U2 MCP3008

Commit message: Updated PCB
Parts:
- J1: footprint Connector_PinHeader_2.54mm:PinHeader_2x20_P2.54mm_Vertical -> Rpi:MODULE_RASPBERRY_PI_3_MODEL_B+
- U1: footprint (none) -> LM2596:LM2596
Changed lines of the file:
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@@
       (effects (font (size 1.27 1.27)) (justify left))
     )
-    (property "Footprint" "Connector_PinHeader_2.54mm:PinHeader_2x20_P2.54mm_Vertical" (at 248.92 87.63 0)
+    (property "Footprint" "Rpi:MODULE_RASPBERRY_PI_3_MODEL_B+" (at 248.92 87.63 0)
       (effects (font (size 1.27 1.27)) hide)
     )
@@
       (effects (font (size 1.27 1.27)))
     )
-    (property "Footprint" "" (at 99.06 97.79 0)
+    (property "Footprint" "LM2596:LM2596" (at 99.06 97.79 0)
       (effects (font (size 1.27 1.27)) hide)
     )

Commit message: final commit
Parts:
- C1: value C -> 90F
- R1: value 1 -> .1
- R2: value 10k -> 100k
Connections:
- net +6V: now also R2.1; no longer U1.3 (-IN)
- net GND: now also U1.3 (-IN)
- net at D1.2 (A), U1.2 (+OUT): no longer R2.1
Other:
- moved on the sheet: R2, R3
Changed lines of the file:
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@@
     (comment 1 "Authors: Alex Santiago-Anaya, Moses Zhou")
   )
-  (junction (at 115.57 96.52) (diameter 0) (color 0 0 0 0)
-  )
   (junction (at 243.84 50.8) (diameter 0) (color 0 0 0 0)
   )
@@
   (junction (at 177.8 88.9) (diameter 0) (color 0 0 0 0)
   )
-  (junction (at 115.57 69.85) (diameter 0) (color 0 0 0 0)
+  (junction (at 76.2 96.52) (diameter 0) (color 0 0 0 0)
+  )
+  (junction (at 81.28 96.52) (diameter 0) (color 0 0 0 0)
   )
   (junction (at 177.8 50.8) (diameter 0) (color 0 0 0 0)
@@
   (junction (at 152.4 67.31) (diameter 0) (color 0 0 0 0)
   )
-  (junction (at 115.57 120.65) (diameter 0) (color 0 0 0 0)
-  )
-  (junction (at 78.74 96.52) (diameter 0) (color 0 0 0 0)
+  (junction (at 81.28 69.85) (diameter 0) (color 0 0 0 0)
   )
   (junction (at 251.46 50.8) (diameter 0) (color 0 0 0 0)
@@
     (stroke (width 0) (type default))
   )
-  (wire (pts (xy 74.93 96.52) (xy 78.74 96.52))
+  (wire (pts (xy 74.93 96.52) (xy 76.2 96.52))
     (stroke (width 0) (type default))
   )
@@
     (stroke (width 0) (type default))
   )
-  (wire (pts (xy 62.23 69.85) (xy 62.23 120.65))
-    (stroke (width 0) (type default))
-  )
-  (wire (pts (xy 62.23 69.85) (xy 104.14 69.85))
+  (wire (pts (xy 81.28 96.52) (xy 82.55 96.52))
+    (stroke (width 0) (type default))
+  )
+  (wire (pts (xy 62.23 69.85) (xy 67.31 69.85))
     (stroke (width 0) (type default))
   )
@@
     (stroke (width 0) (type default))
   )
-  (wire (pts (xy 115.57 96.52) (xy 116.84 96.52))
+  (wire (pts (xy 74.93 69.85) (xy 81.28 69.85))
     (stroke (width 0) (type default))
   )
@@
     (stroke (width 0) (type default))
   )
-  (wire (pts (xy 62.23 120.65) (xy 115.57 120.65))
-    (stroke (width 0) (type default))
-  )
-  (wire (pts (xy 110.49 96.52) (xy 115.57 96.52))
-    (stroke (width 0) (type default))
-  )
   (wire (pts (xy 170.18 88.9) (xy 177.8 88.9))
     (stroke (width 0) (type default))
@@
     (stroke (width 0) (type default))
   )
+  (wire (pts (xy 81.28 69.85) (xy 157.48 69.85))
+    (stroke (width 0) (type default))
+  )
   (wire (pts (xy 170.18 50.8) (xy 177.8 50.8))
     (stroke (width 0) (type default))
@@
     (stroke (width 0) (type default))
   )
-  (wire (pts (xy 115.57 81.28) (xy 115.57 96.52))
+  (wire (pts (xy 81.28 82.55) (xy 81.28 96.52))
     (stroke (width 0) (type default))
   )
@@
     (stroke (width 0) (type default))
   )
-  (wire (pts (xy 115.57 73.66) (xy 115.57 69.85))
+  (wire (pts (xy 81.28 74.93) (xy 81.28 69.85))
     (stroke (width 0) (type default))
   )
@@
     (stroke (width 0) (type default))
   )
-  (wire (pts (xy 78.74 96.52) (xy 82.55 96.52))
-    (stroke (width 0) (type default))
-  )
   (wire (pts (xy 170.18 87.63) (xy 170.18 88.9))
     (stroke (width 0) (type default))
@@
     (stroke (width 0) (type default))
   )
-  (wire (pts (xy 115.57 69.85) (xy 157.48 69.85))
-    (stroke (width 0) (type default))
-  )
   (wire (pts (xy 187.96 74.93) (xy 212.09 74.93))
     (stroke (width 0) (type default))
@@
     (stroke (width 0) (type default))
   )
+  (wire (pts (xy 110.49 96.52) (xy 116.84 96.52))
+    (stroke (width 0) (type default))
+  )
   (wire (pts (xy 187.96 69.85) (xy 217.17 69.85))
     (stroke (width 0) (type default))
   )
-  (wire (pts (xy 111.76 69.85) (xy 115.57 69.85))
+  (wire (pts (xy 76.2 96.52) (xy 81.28 96.52))
     (stroke (width 0) (type default))
   )
@@
     (stroke (width 0) (type default))
   )
-  (wire (pts (xy 78.74 93.98) (xy 78.74 96.52))
+  (wire (pts (xy 76.2 93.98) (xy 76.2 96.52))
     (stroke (width 0) (type default))
   )
@@
     )
   )
-  (symbol (lib_id "power:+6V") (at 74.93 102.87 90) (unit 1)
-    (in_bom yes) (on_board yes) (dnp no)
-    (property "Reference" "#PWR03" (at 78.74 102.87 0)
-      (effects (font (size 1.27 1.27)) hide)
-    )
-    (property "Value" "0V" (at 71.12 103.505 90)
-      (effects (font (size 1.27 1.27)) (justify left))
-    )
-    (property "Footprint" "" (at 74.93 102.87 0)
-      (effects (font (size 1.27 1.27)) hide)
-    )
-    (property "Datasheet" "" (at 74.93 102.87 0)
-      (effects (font (size 1.27 1.27)) hide)
-    )
-    (pin "1")
-    (instances
-      (project "scm-pcb"
-        (path "/d592ecb6-f86c-47c7-8da3-aafda8863a2e"
-          (reference "#PWR03") (unit 1)
-        )
-      )
-    )
-  )
-  (symbol (lib_id "power:PWR_FLAG") (at 78.74 93.98 0) (unit 1)
-    (in_bom yes) (on_board yes) (dnp no) (fields_autoplaced)
-    (property "Reference" "#FLG01" (at 78.74 92.075 0)
-      (effects (font (size 1.27 1.27)) hide)
-    )
-    (property "Value" "PWR_FLAG" (at 78.74 90.17 0)
-      (effects (font (size 1.27 1.27)))
-    )
-    (property "Footprint" "" (at 78.74 93.98 0)
-      (effects (font (size 1.27 1.27)) hide)
-    )
-    (property "Datasheet" "~" (at 78.74 93.98 0)
+  (symbol (lib_id "power:GND") (at 62.23 69.85 0) (unit 1)
+    (in_bom yes) (on_board yes) (dnp no) (fields_autoplaced)
+    (property "Reference" "#PWR04" (at 62.23 76.2 0)
+      (effects (font (size 1.27 1.27)) hide)
+    )
+    (property "Value" "GND" (at 62.23 74.93 0)
+      (effects (font (size 1.27 1.27)))
+    )
+    (property "Footprint" "" (at 62.23 69.85 0)
+      (effects (font (size 1.27 1.27)) hide)
+    )
+    (property "Datasheet" "" (at 62.23 69.85 0)
+      (effects (font (size 1.27 1.27)) hide)
+    )
+    (pin "1")
+    (instances
+      (project "scm-pcb"
+        (path "/d592ecb6-f86c-47c7-8da3-aafda8863a2e"
+          (reference "#PWR04") (unit 1)
+        )
+      )
+    )
+  )
+  (symbol (lib_id "power:PWR_FLAG") (at 76.2 93.98 0) (unit 1)
+    (in_bom yes) (on_board yes) (dnp no) (fields_autoplaced)
+    (property "Reference" "#FLG01" (at 76.2 92.075 0)
+      (effects (font (size 1.27 1.27)) hide)
+    )
+    (property "Value" "PWR_FLAG" (at 76.2 90.17 0)
+      (effects (font (size 1.27 1.27)))
+    )
+    (property "Footprint" "" (at 76.2 93.98 0)
+      (effects (font (size 1.27 1.27)) hide)
+    )
+    (property "Datasheet" "~" (at 76.2 93.98 0)
       (effects (font (size 1.27 1.27)) hide)
     )
@@
     )
   )
-  (symbol (lib_id "Device:R") (at 107.95 69.85 90) (unit 1)
-    (in_bom yes) (on_board yes) (dnp no) (fields_autoplaced)
-    (property "Reference" "R3" (at 107.95 64.77 90)
-      (effects (font (size 1.27 1.27)))
-    )
-    (property "Value" "10k" (at 107.95 67.31 90)
-      (effects (font (size 1.27 1.27)))
-    )
-    (property "Footprint" "Resistors:CMF5510K000FKEB" (at 107.95 71.628 90)
-      (effects (font (size 1.27 1.27)) hide)
-    )
-    (property "Datasheet" "~" (at 107.95 69.85 0)
+  (symbol (lib_id "Device:R") (at 71.12 69.85 90) (unit 1)
+    (in_bom yes) (on_board yes) (dnp no) (fields_autoplaced)
+    (property "Reference" "R3" (at 71.12 64.77 90)
+      (effects (font (size 1.27 1.27)))
+    )
+    (property "Value" "10k" (at 71.12 67.31 90)
+      (effects (font (size 1.27 1.27)))
+    )
+    (property "Footprint" "Resistors:CMF5510K000FKEB" (at 71.12 71.628 90)
+      (effects (font (size 1.27 1.27)) hide)
+    )
+    (property "Datasheet" "~" (at 71.12 69.85 0)
       (effects (font (size 1.27 1.27)) hide)
     )
@@
     )
   )
-  (symbol (lib_id "Device:R") (at 115.57 77.47 180) (unit 1)
-    (in_bom yes) (on_board yes) (dnp no) (fields_autoplaced)
-    (property "Reference" "R2" (at 118.11 76.835 0)
+  (symbol (lib_id "Device:R") (at 81.28 78.74 180) (unit 1)
+    (in_bom yes) (on_board yes) (dnp no) (fields_autoplaced)
+    (property "Reference" "R2" (at 83.82 78.105 0)
       (effects (font (size 1.27 1.27)) (justify right))
     )
-    (property "Value" "10k" (at 118.11 79.375 0)
+    (property "Value" "100k" (at 83.82 80.645 0)
       (effects (font (size 1.27 1.27)) (justify right))
     )
-    (property "Footprint" "Resistors:CMF5510K000FKEB" (at 117.348 77.47 90)
-      (effects (font (size 1.27 1.27)) hide)
-    )
-    (property "Datasheet" "~" (at 115.57 77.47 0)
+    (property "Footprint" "Resistors:CMF5510K000FKEB" (at 83.058 78.74 90)
+      (effects (font (size 1.27 1.27)) hide)
+    )
+    (property "Datasheet" "~" (at 81.28 78.74 0)
       (effects (font (size 1.27 1.27)) hide)
     )
@@
       (effects (font (size 1.27 1.27)) (justify left))
     )
-    (property "Value" "C" (at 135.89 111.125 0)
+    (property "Value" "90F" (at 135.89 111.125 0)
       (effects (font (size 1.27 1.27)) (justify left))
     )
@@
     )
   )
+  (symbol (lib_id "power:GND") (at 74.93 102.87 0) (unit 1)
+    (in_bom yes) (on_board yes) (dnp no) (fields_autoplaced)
+    (property "Reference" "#PWR03" (at 74.93 109.22 0)
+      (effects (font (size 1.27 1.27)) hide)
+    )
+    (property "Value" "GND" (at 74.93 107.95 0)
+      (effects (font (size 1.27 1.27)))
+    )
+    (property "Footprint" "" (at 74.93 102.87 0)
+      (effects (font (size 1.27 1.27)) hide)
+    )
+    (property "Datasheet" "" (at 74.93 102.87 0)
+      (effects (font (size 1.27 1.27)) hide)
+    )
+    (pin "1")
+    (instances
+      (project "scm-pcb"
+        (path "/d592ecb6-f86c-47c7-8da3-aafda8863a2e"
+          (reference "#PWR03") (unit 1)
+        )
+      )
+    )
+  )
   (symbol (lib_id "Device:R") (at 135.89 96.52 90) (unit 1)
     (in_bom yes) (on_board yes) (dnp no) (fields_autoplaced)
@@
       (effects (font (size 1.27 1.27)))
     )
-    (property "Value" "1" (at 135.89 93.98 90)
-      (effects (font (size 1.27 1.27)))
-    )
+    (property "Value" ".1" (at 135.89 93.98 90)
+      (effects (font (size 1.27 1.27)))
+    )
